File: ddr4-dimm-test.kicad_sch (KiCad schematic)
At the start: 150 parts

Commit message: there's a ddr5 dimm symbol too now
felt like making it, for future use i guess
Parts:
- added GF2: DDR5-dimm-edge, symbol A-my-stuff:DDR5-dimm-edge
